Commit message: changed to 5 joints

File: src/yannic/yannic_robot/urdf/yannic_robot.urdf (robot description, URDF)
Before this commit: robot yannic_robot, 7 links, 6 joints
Links:
- added link endeff, mass 0.01; collision box size=0.0001 0.001 0.01; visual box size=0.0001 0.001 0.01
Joints:
- added joint endeff_joint: type fixed, parent link3, child endeff, origin xyz=0.054 0 0 rpy=0 0 0

File: src/yannic/yannic_robot/urdf/yannic_robot.urdf.xacro (robot description, xacro)
@@ -173,3 +173,23 @@
     <xacro:default_inertial mass="0.5"/>
    </link>
+   <joint name="endeff_joint" type="fixed">
+     <origin rpy="0 0 0" xyz="${link3_length} 0 0"/>
+     <parent link="link3"/>
+     <child link="endeff"/>
+   </joint>
+   <link name="endeff">
+   <visual>
+      <geometry>
+         <box size="0.0001 ${width}  ${length}"/>
+      </geometry>
+      <material name="transparent"/>
+      <origin rpy="0 0 0" xyz="${0.0001/2} 0 0.0"/>
+    </visual>
+	    <collision>
+      <geometry>
+        <box size="0.0001 ${width}  ${length}"/>
+      </geometry>
+    </collision>
+   <xacro:default_inertial mass="0.01"/>
+   </link>
 </robot>
